File: hardware/picoBuck.brd (EAGLE design)
At the start: 36.2 x 29.8 mm, 37 parts, among them U1 AL8805WS, U2 AL8805WS, U3 AL8805WS

Commit message: Fixed issues from qc feedback
Parts:
- removed CH2, CH3: (no value), SparkFun:SCREWTERMINAL-3.5MM-2_LOCK
- added JP5: M022.54MM_SCREWTERM, SparkFun-Connectors:1X02_2.54_SCREWTERM
- added JP6: (no value), SparkFun:SCREWTERMINAL-3.5MM-2_LOCK
- JP3: value M022.54MM_SCREWTERM -> (none); device SparkFun-Connectors:1X02_2.54_SCREWTERM -> SparkFun:SCREWTERMINAL-3.5MM-2_LOCK
- moved JP2 25.3 mm to (11.0, 2.54), turned to 0 degrees
- moved JP3 24.2 mm to (19.7, 2.54)
- moved JP4 7.62 mm to (21.0, 26.7)
- renumbered CH1 to JP1
Connections:
- net CTRL_CH1: now also JP5.P1; no longer JP4.P1
- net CTRL_CH2: now also JP4.P2; no longer JP3.P2
- net CTRL_CH3: now also JP4.P1; no longer JP3.P1
- net GND: now also JP5.P2, JP6.1; no longer JP2.1, JP4.P2
- net N$1: now also JP3.1; no longer CH3.1
- net N$13: now also JP2.1; no longer CH2.1
- net N$16: now also JP3.2; no longer CH3.2
- net N$9: now also JP2.2; no longer CH2.2
- net VIN: now also JP6.2; no longer JP2.2
Other:
- board text added: "SJ1"
- board text added: "SJ2"
- board text added: "SJ3"
Changed lines of the file:
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@@
 <text x="34.544" y="6.731" size="1.778" layer="47" font="vector" ratio="15">#4-40 typ.</text>
 <text x="2.54" y="-19.05" size="1.778" layer="47" font="vector" ratio="15">Units are inches</text>
+<text x="1.778" y="21.971" size="0.8128" layer="21" font="vector" ratio="15" rot="R90" align="bottom-center">SJ1</text>
+<text x="10.414" y="21.971" size="0.8128" layer="21" font="vector" ratio="15" rot="R90" align="bottom-center">SJ2</text>
+<text x="19.05" y="21.971" size="0.8128" layer="21" font="vector" ratio="15" rot="R90" align="bottom-center">SJ3</text>
 </plain>
 <attributes>
@@
 <param name="rlMinPadBottom" value="12mil"/>
 <param name="rlMaxPadBottom" value="20mil"/>
-<param name="rlMinViaOuter" value="7mil"/>
+<param name="rlMinViaOuter" value="10mil"/>
 <param name="rlMaxViaOuter" value="20mil"/>
-<param name="rlMinViaInner" value="7mil"/>
+<param name="rlMinViaInner" value="10mil"/>
 <param name="rlMaxViaInner" value="20mil"/>
 <param name="rlMinMicroViaOuter" value="4mil"/>
@@
 <attribute name="VALUE" value="33uH" x="22.225" y="10.668" size="1.778" layer="27" display="off"/>
 </element>
-<element name="JP2" library="SparkFun" package="SCREWTERMINAL-3.5MM-2_LOCK" value="" x="5.87375" y="27.305" rot="R180"/>
-<element name="CH2" library="SparkFun" package="SCREWTERMINAL-3.5MM-2_LOCK" value="" x="11.049" y="2.54"/>
-<element name="CH1" library="SparkFun" package="SCREWTERMINAL-3.5MM-2_LOCK" value="" x="2.413" y="2.54"/>
-<element name="CH3" library="SparkFun" package="SCREWTERMINAL-3.5MM-2_LOCK" value="" x="19.685" y="2.54"/>
+<element name="JP6" library="SparkFun" package="SCREWTERMINAL-3.5MM-2_LOCK" value="" x="5.87375" y="27.305" rot="R180"/>
+<element name="JP2" library="SparkFun" package="SCREWTERMINAL-3.5MM-2_LOCK" value="" x="11.049" y="2.54"/>
+<element name="JP1" library="SparkFun" package="SCREWTERMINAL-3.5MM-2_LOCK" value="" x="2.413" y="2.54"/>
+<element name="JP3" library="SparkFun" package="SCREWTERMINAL-3.5MM-2_LOCK" value="" x="19.685" y="2.54"/>
 <element name="C5" library="SparkFun-Capacitors" package="0805-CAP" value="1.0uF" x="24.892" y="16.3195" rot="R270">
 <attribute name="PROD_ID" value="CAP-11625" x="24.892" y="16.3195" size="1.778" layer="27" rot="R270" display="off"/>
@@
 <element name="LOGO2" library="SparkFun-Aesthetics" package="SFE-NEW-WEBLOGO" value="LOGO-SFENEW" x="23.241" y="3.429" rot="MR0"/>
 <element name="FRAME1" library="SparkFun-Aesthetics" package="CREATIVE_COMMONS" value="FRAME-LETTER" x="11.43" y="-31.75"/>
-<element name="JP3" library="SparkFun-Connectors" package="1X02_2.54_SCREWTERM" value="M022.54MM_SCREWTERM" x="20.955" y="26.67"/>
-<element name="JP4" library="SparkFun-Connectors" package="1X02_2.54_SCREWTERM" value="M022.54MM_SCREWTERM" x="13.335" y="26.67"/>
+<element name="JP4" library="SparkFun-Connectors" package="1X02_2.54_SCREWTERM" value="M022.54MM_SCREWTERM" x="20.955" y="26.67"/>
+<element name="JP5" library="SparkFun-Connectors" package="1X02_2.54_SCREWTERM" value="M022.54MM_SCREWTERM" x="13.335" y="26.67"/>
 <element name="FID1" library="SparkFun-Aesthetics" package="MICRO-FIDUCIAL" value="FIDUCIALUFIDUCIAL" x="4.318" y="1.016"/>
 <element name="FID2" library="SparkFun-Aesthetics" package="MICRO-FIDUCIAL" value="FIDUCIALUFIDUCIAL" x="24.003" y="28.448"/>
@@
 <contactref element="U3" pad="2"/>
 <contactref element="C6" pad="2"/>
-<contactref element="JP2" pad="1"/>
+<contactref element="JP6" pad="1"/>
 <polygon width="0.254" layer="16" isolate="0.3048">
 <vertex x="0.0254" y="29.8196"/>
@@
 <vertex x="0" y="0"/>
 </polygon>
-<contactref element="JP4" pad="P2"/>
+<contactref element="JP5" pad="P2"/>
 <wire x1="7.62" y1="20.055" x2="7.62" y2="18.542" width="0.8128" layer="1"/>
 <via x="7.62" y="18.542" extent="1-16" drill="0.381"/>
@@
 <contactref element="U3" pad="5"/>
 <contactref element="C6" pad="1"/>
-<contactref element="JP2" pad="2"/>
-<polygon width="0.254" layer="1" isolate="0.2032" rank="2">
+<contactref element="JP6" pad="2"/>
+<polygon width="0.254" layer="1" isolate="0.254" rank="2">
 <vertex x="0.635" y="28.8925"/>
 <vertex x="3.81" y="28.8925"/>
@@
 <contactref element="C3" pad="2"/>
 <contactref element="L2" pad="2"/>
-<contactref element="CH2" pad="2"/>
+<contactref element="JP2" pad="2"/>
 <polygon width="0.254" layer="1" isolate="0.2032" rank="3">
 <vertex x="15.621" y="17.145"/>
@@
 </signal>
 <signal name="N$13">
-<contactref element="CH2" pad="1"/>
+<contactref element="JP2" pad="1"/>
 <contactref element="R2" pad="2"/>
 <contactref element="R5" pad="1"/>
@@
 <contactref element="C1" pad="2"/>
 <contactref element="L1" pad="2"/>
-<contactref element="CH1" pad="2"/>
+<contactref element="JP1" pad="2"/>
 <polygon width="0.254" layer="1" isolate="0.2032" rank="3">
 <vertex x="6.985" y="17.145"/>
@@
 </signal>
 <signal name="N$11">
-<contactref element="CH1" pad="1"/>
+<contactref element="JP1" pad="1"/>
 <contactref element="R4" pad="1"/>
 <contactref element="R1" pad="2"/>
@@
 <signal name="N$16" class="1">
 <contactref element="L3" pad="2"/>
-<contactref element="CH3" pad="2"/>
+<contactref element="JP3" pad="2"/>
 <contactref element="C5" pad="2"/>
 <polygon width="0.254" layer="1" isolate="0.2032" rank="3">
@@
 <signal name="CTRL_CH1">
 <contactref element="U1" pad="3"/>
-<contactref element="JP4" pad="P1"/>
+<contactref element="JP5" pad="P1"/>
 <wire x1="5.903" y1="15.8449" x2="5.903" y2="14.544" width="0.2032" layer="1"/>
 <wire x1="5.903" y1="14.544" x2="6.096" y2="14.351" width="0.2032" layer="1"/>
@@
 <signal name="CTRL_CH2">
 <contactref element="U2" pad="3"/>
-<contactref element="JP3" pad="P2"/>
+<contactref element="JP4" pad="P2"/>
 <wire x1="14.539" y1="15.8449" x2="14.539" y2="14.544" width="0.2032" layer="1"/>
 <wire x1="14.539" y1="14.544" x2="14.732" y2="14.351" width="0.2032" layer="1"/>
@@
 <signal name="CTRL_CH3">
 <contactref element="U3" pad="3"/>
-<contactref element="JP3" pad="P1"/>
+<contactref element="JP4" pad="P1"/>
 <wire x1="23.175" y1="15.8449" x2="23.175" y2="14.671" width="0.2032" layer="1"/>
 <wire x1="23.175" y1="14.671" x2="23.495" y2="14.351" width="0.2032" layer="1"/>
@@
 <contactref element="C5" pad="1"/>
 <contactref element="R6" pad="1"/>
-<contactref element="CH3" pad="1"/>
+<contactref element="JP3" pad="1"/>
 <contactref element="R3" pad="2"/>
 <polygon width="0.2032" layer="1" isolate="0.2032">
